File: hardware/weather-featherwing.kicad_pcb (KiCad board)
At the start: 2 copper layers, 50.8 x 22.9 mm, 35 parts, among them J1 Feather_Header_01x16, J2 Feather_Header_01x12, J3 MEM2061, J4 STEMMA-QT, SW1 JS102011SAQN, U1 LPS22HB, U2 SHT41, U3 11AA010

Commit message: 1.2.1 changes
Parts:
- added FID3: Fiducial, lib_fp:Fiducial_1mm_Mask2mm, F.Cu at (119.7, 102.4)
- U1: footprint DS-Master-Sensors-SMD:PQFN10P50_200X200X80L27X25N -> lib_fp:LPS22
Connections:
- J4 pad 1: (no net) -> GND
- J4 pad 3: (no net) -> /SDA
- J4 pad 4: (no net) -> /SCL
- J4 pad MP: (no net) -> GND
- SW1 pad 1: unconnected-(SW1-A-Pad1) -> /EN
- SW1 pad 3: /EN -> unconnected-(SW1-C-Pad3)
Routing:
- net /EN: track 15.5 -> 7.84 mm
- net unconnected-(SW1-C-Pad3): track 0.00 -> 1.25 mm
- net GND: vias 60 -> 59
Other:
- board text added: "Weather FeatherWing v1.2.1 2024-02-19"
- board text removed: "Weather FeatherWing v1.2.0 2024-01-28"
