File: hardware/weather-featherwing.kicad_sch (KiCad schematic)
At the start: 32 parts, among them J1 Feather_Header_01x16, J2 Feather_Header_01x12, J3 MEM2061, J4 STEMMA-QT, SW1 JS102011SAQN, U1 LPS22HB, U2 SHT41, U3 11AA010

Commit message: 1.2.1 changes
Parts:
- added FID3: Fiducial, lib_fp:Fiducial_1mm_Mask2mm, symbol lib_sch:Fiducial
- U1: footprint DS-Master-Sensors-SMD:PQFN10P50_200X200X80L27X25N -> lib_fp:LPS22
Connections:
- net EN: now also SW1.1 (A); no longer SW1.3 (C)
Other:
- title: Weather Featherwing v1.1.0 -> Weather Featherwing v1.2.1
- moved on the sheet: FID1, FID2, SW1
Changed lines of the file:
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@@
   (paper "USLetter")
   (title_block
-    (title "Weather Featherwing v1.1.0")
-    (date "2024-01-07")
+    (title "Weather Featherwing v1.2.1")
+    (date "2024-02-19")
     (rev "02")
     (comment 1 "Madison Gleydura")
@@
       (effects (font (size 1.27 1.27)) (justify left top))
     )
-    (property "Footprint" "DS-Master-Sensors-SMD:PQFN10P50_200X200X80L27X25N" (at 63.5 114.3 0)
+    (property "Footprint" "lib_fp:LPS22" (at 63.5 114.3 0)
       (effects (font (size 1.27 1.27)) hide)
     )
@@
     )
   )
-  (symbol (lib_id "lib_sch:SW_SPDT") (at 76.2 33.02 270) (mirror x) (unit 1)
-    (in_bom yes) (on_board yes) (dnp no)
-    (property "Reference" "SW1" (at 81.28 34.29 90) (do_not_autoplace)
+  (symbol (lib_id "lib_sch:SW_SPDT") (at 76.2 33.02 90) (unit 1)
+    (in_bom yes) (on_board yes) (dnp no)
+    (property "Reference" "SW1" (at 71.12 34.29 90) (do_not_autoplace)
       (effects (font (size 1.27 1.27)) (justify left))
     )
-    (property "Value" "JS102011SAQN" (at 81.28 31.75 90) (do_not_autoplace)
+    (property "Value" "JS102011SAQN" (at 71.12 31.75 90) (do_not_autoplace)
       (effects (font (size 1.27 1.27)) (justify left))
     )
@@
     )
   )
+  (symbol (lib_id "lib_sch:Fiducial") (at 57.15 57.15 0) (mirror y) (unit 1)
+    (in_bom no) (on_board yes) (dnp yes) (fields_autoplaced)
+    (property "Reference" "FID3" (at 54.61 55.88 0)
+      (effects (font (size 1.27 1.27)) (justify left))
+    )
+    (property "Value" "Fiducial" (at 54.61 58.42 0)
+      (effects (font (size 1.27 1.27)) (justify left))
+    )
+    (property "Footprint" "lib_fp:Fiducial_1mm_Mask2mm" (at 57.15 57.15 0)
+      (effects (font (size 1.27 1.27)) hide)
+    )
+    (property "Datasheet" "~" (at 57.15 57.15 0)
+      (effects (font (size 1.27 1.27)) hide)
+    )
+    (property "Manufacturer" "~" (at 57.15 57.15 0)
+      (effects (font (size 1.27 1.27)) hide)
+    )
+    (property "mpn" "~" (at 57.15 57.15 0)
+      (effects (font (size 1.27 1.27)) hide)
+    )
+    (property "populate" "0" (at 57.15 57.15 0)
+      (effects (font (size 1.27 1.27)) hide)
+    )
+    (instances
+      (project "weather-featherwing"
+        (path "/3087481e-f72d-4c6b-8051-de7bcae4a5de"
+          (reference "FID3") (unit 1)
+        )
+      )
+    )
+  )
   (symbol (lib_id "lib_sch:r_small") (at 191.77 21.59 0) (unit 1)
     (in_bom yes) (on_board yes) (dnp no) (fields_autoplaced)
@@
     )
   )
-  (symbol (lib_id "lib_sch:Fiducial") (at 57.15 57.15 0) (mirror y) (unit 1)
+  (symbol (lib_id "lib_sch:Fiducial") (at 57.15 52.07 0) (mirror y) (unit 1)
     (in_bom no) (on_board yes) (dnp yes) (fields_autoplaced)
-    (property "Reference" "FID2" (at 54.61 55.88 0)
+    (property "Reference" "FID2" (at 54.61 50.8 0)
       (effects (font (size 1.27 1.27)) (justify left))
     )
-    (property "Value" "Fiducial" (at 54.61 58.42 0)
+    (property "Value" "Fiducial" (at 54.61 53.34 0)
       (effects (font (size 1.27 1.27)) (justify left))
     )
-    (property "Footprint" "lib_fp:Fiducial_1mm_Mask2mm" (at 57.15 57.15 0)
-      (effects (font (size 1.27 1.27)) hide)
-    )
-    (property "Datasheet" "~" (at 57.15 57.15 0)
-      (effects (font (size 1.27 1.27)) hide)
-    )
-    (property "Manufacturer" "~" (at 57.15 57.15 0)
-      (effects (font (size 1.27 1.27)) hide)
-    )
-    (property "mpn" "~" (at 57.15 57.15 0)
-      (effects (font (size 1.27 1.27)) hide)
-    )
-    (property "populate" "0" (at 57.15 57.15 0)
+    (property "Footprint" "lib_fp:Fiducial_1mm_Mask2mm" (at 57.15 52.07 0)
+      (effects (font (size 1.27 1.27)) hide)
+    )
+    (property "Datasheet" "~" (at 57.15 52.07 0)
+      (effects (font (size 1.27 1.27)) hide)
+    )
+    (property "Manufacturer" "~" (at 57.15 52.07 0)
+      (effects (font (size 1.27 1.27)) hide)
+    )
+    (property "mpn" "~" (at 57.15 52.07 0)
+      (effects (font (size 1.27 1.27)) hide)
+    )
+    (property "populate" "0" (at 57.15 52.07 0)
       (effects (font (size 1.27 1.27)) hide)
     )
@@
     )
   )
-  (symbol (lib_id "lib_sch:Fiducial") (at 57.15 52.07 0) (mirror y) (unit 1)
+  (symbol (lib_id "lib_sch:Fiducial") (at 57.15 46.99 0) (mirror y) (unit 1)
     (in_bom no) (on_board yes) (dnp yes) (fields_autoplaced)
-    (property "Reference" "FID1" (at 54.61 50.8 0)
+    (property "Reference" "FID1" (at 54.61 45.72 0)
       (effects (font (size 1.27 1.27)) (justify left))
     )
-    (property "Value" "Fiducial" (at 54.61 53.34 0)
+    (property "Value" "Fiducial" (at 54.61 48.26 0)
       (effects (font (size 1.27 1.27)) (justify left))
     )
-    (property "Footprint" "lib_fp:Fiducial_1mm_Mask2mm" (at 57.15 52.07 0)
-      (effects (font (size 1.27 1.27)) hide)
-    )
-    (property "Datasheet" "~" (at 57.15 52.07 0)
-      (effects (font (size 1.27 1.27)) hide)
-    )
-    (property "Manufacturer" "~" (at 57.15 52.07 0)
-      (effects (font (size 1.27 1.27)) hide)
-    )
-    (property "mpn" "~" (at 57.15 52.07 0)
-      (effects (font (size 1.27 1.27)) hide)
-    )
-    (property "populate" "0" (at 57.15 52.07 0)
-      (effects (font (size 1.27 1.27)) hide)
-    )
+    (property "Footprint" "lib_fp:Fiducial_1mm_Mask2mm" (at 57.15 46.99 0)
+      (effects (font (size 1.27 1.27)) hide)
+    )
+    (property "Datasheet" "~" (at 57.15 46.99 0)
+      (effects (font (size 1.27 1.27)) hide)
+    )
+    (property "Manufacturer" "~" (at 57.15 46.99 0)
+      (effects (font (size 1.27 1.27)) hide)
+    )
+    (property "mpn" "~" (at 57.15 46.99 0)
+      (effects (font (size 1.27 1.27)) hide)
+    )
+    (property "populate" "0" (at 57.15 46.99 0)
+      (effects (font (size 1.27 1.27)) hide)
+    )
