File: hardware/weather-featherwing/weather-featherwing.kicad_pcb (KiCad board)
At the start: 2 copper layers, 50.8 x 22.9 mm, 36 parts, among them J1 Feather_Header_01x16, J2 Feather_Header_01x12, J3 MEM2061, J4 STEMMA-QT, SW1 JS102011SAQN, U1 LPS22HB, U2 SHT41, U3 11AA010

Commit message: rev3 changes
Other:
- outline, holes or cut-outs redrawn
- board text added: "Weather FeatherWing v1.2.2 2024-03-09"
- board text removed: "Weather FeatherWing v1.2.1 2024-02-19"

Commit message: blender renders and cleaned up files
Parts:
- moved FID2 0.15 mm to (119.7, 114.9)
Routing:
- net +3V3: track 83.1 -> 84.0 mm
- net GND: vias 59 -> 65
Other:
- board text added: "PCB3D_BR_Weather-FeatherWing"
- board text added: "Weather FeatherWing v1.2.2 2024-03-10"
- board text removed: "Weather FeatherWing v1.2.2 2024-03-09"

Commit message: housekeeping
Parts:
- U2: footprint DS-Master-Sensors-SMD:SHT4x -> lib_fp:SHT4x
Routing:
- net GND: vias 65 -> 63
