File: hardware/weather-featherwing/weather-featherwing.kicad_pcb (KiCad board)
At the start: 2 copper layers, 50.8 x 22.9 mm, 36 parts, among them J1 Feather_Header_01x16, J2 Feather_Header_01x12, J3 MEM2061, J4 STEMMA-QT, SW1 JS102011SAQN, U1 LPS22HB, U2 SHT41, U3 11AA010

Commit message: organization
Other:
- board text added: "Weather FeatherWing v1.2.2 2024-03-26"
- board text removed: "Weather FeatherWing v1.2.2 2024-03-10"
